File: Hardware/Kicad/lps_regulator/lps_regulator_rev_12.kicad_pcb (KiCad board)
At the start: 2 copper layers, 136.2 x 62.6 mm, 135 parts, among them CN1 Header 5X2A, CN2 Header 8X2A, CN3 Header 2H, CN4 Header 2H, CN5 Header 2H, Q1 MMBT2907A, Q2 MMBT3904, Q3 MMBT3904, Q4 BSS123TA, Q5 MMBT2907A, Q6 BSS123TA, U1 TPS7A4515KTTR, U11 LD1117S33, U12 LM2776, U14 TPS54331, U2 INA180A1, U3 INA219, U4 OPA2320, U5 LM334, U6 mcp9808, U7 mcp4728, U8 TCA9534APWR, U9 OPA2320

Commit message: Add files via upload
Parts:
- removed C22: 10uF, Vault:CAPC0603(1608)_N
- moved C23 0.11 mm to (95.8, 107.2)
- renumbered C27 to C17, C17 to C51, C24 to C60
Routing:
- net GND: track 55.1 -> 60.0 mm, vias 4 -> 35
- net +5V0: track 39.2 -> 37.8 mm
- net NetC47_2: track 22.4 -> 23.4 mm
- net I2C_SDA: track 166.0 -> 165.2 mm
- net NetQ2_1: track 4.11 -> 3.56 mm
Other:
- board text added: "Debug Led"
