File: Hardware/Kicad/lps_regulator/lps_regulator_rev_12.kicad_sch (KiCad schematic)
At the start: 133 parts, among them CN1 Header 2H, CN2 Header 8X2A, CN3 Header 2H, CN4 Header 2H, CN5 Header 5X2A, Q1 MMBT2907A, Q2 MMBT2907A, Q3 MMBT3904, Q4 MMBT3904, Q5 BSS123TA, Q6 BSS123TA, U10 TPS7A4515KTTR, U11 OPA2320, U12 OPA2320, U13 INA219, U14 INA180A1, U15 LM334, U2 mcp4728, U3 TPS54331, U4 mcp9808, U5 LD1117S33, U6 OPA2320, U7 TCA9534APWR, U8 LM2776, U9 OPA2320

Commit message: Add files via upload
Parts:
- removed +5V1, -5V1, 3V1, GND1, GND2, GND3, GND4, IA_TP1, OSA_TP1, REG_IN1, Spare_1, VA_TP1: TestPoint_BLK, TestPoint-TH 42 mil, symbol OLogic Nexus Vault:root_3_TestPoint_BLK_OLogic Nexus Vault
- removed +VIN_SW1, I2C_SCL1, I2C_SDA1, I_sample1, TP1, TP2: TestPoint_BLK, TestPoint-TH 42 mil, symbol OLogic Nexus Vault:root_1_TestPoint_BLK_OLogic Nexus Vault
- removed C1, C2: 4.7uF, CAPC1206(3216)_N, symbol OLogic Nexus Vault:root_3_=Capacitance_OLogic Nexus Vault_1
- removed C10, C19, C22, C35, C38, C8: 0.1uF, CAPC0603(1608)_N, symbol OLogic Nexus Vault:root_0_=Capacitance_OLogic Nexus Vault_1
- removed C11, C17, C23, C25, C29, C30, C37, C41, C42, C44: 10uF, CAPC0603(1608)_N, symbol OLogic Nexus Vault:root_3_=Capacitance_OLogic Nexus Vault_1
- removed C12, C16, C21, C27, C31, C36, C39, C40, C45, C46, C9: 0.1uF, CAPC0603(1608)_N, symbol OLogic Nexus Vault:root_3_=Capacitance_OLogic Nexus Vault_1
- removed C13, C15: 47UF, CAPC1206(3216)_N, symbol OLogic Nexus Vault:root_3_=Capacitance_OLogic Nexus Vault_1
- removed C14, C20, C32: 0.1uF, CAPC0603(1608)_N, symbol OLogic Nexus Vault:root_2_=Capacitance_OLogic Nexus Vault_1
- removed C18: 100pF, CAPC0603(1608)_N, symbol OLogic Nexus Vault:root_0_=Capacitance_OLogic Nexus Vault_1
- removed C24, C6: 1uF, CAPC0603(1608)_N, symbol OLogic Nexus Vault:root_3_=Capacitance_OLogic Nexus Vault_1
- removed C26, C34: 10uF, CAPC0603(1608)_N, symbol OLogic Nexus Vault:root_2_=Capacitance_OLogic Nexus Vault_1
- removed C28: 10uF, CAPC0603(1608)_N, symbol OLogic Nexus Vault:root_0_=Capacitance_OLogic Nexus Vault_1
- removed C3, C5: 0.01uF, CAPC0603(1608)_N, symbol OLogic Nexus Vault:root_3_=Capacitance_OLogic Nexus Vault_1
- removed C33: 1uF, CAPC0603(1608)_N, symbol OLogic Nexus Vault:root_1_=Capacitance_OLogic Nexus Vault_1
- removed C4: 150pF, CAPC0603(1608)_N, symbol OLogic Nexus Vault:root_3_=Capacitance_OLogic Nexus Vault_1
- removed C43: 0.1uF, CAPC0603(1608)_M, symbol OLogic Nexus Vault:root_3_=Capacitance_OLogic Nexus Vault_1
- removed C7: 8.2nf, CAPC1608X87X35ML15T15, symbol OLogic Nexus Vault:root_1_CAP_OLogic Nexus Vault_0
- removed CN1: Header 2H, HDR1X2H, symbol OLogic Nexus Vault:root_0_mirrored_Header 2H_OLogic Nexus Vault
- removed CN2: Header 8X2A, HDR2X8_CEN, symbol OLogic Nexus Vault:root_0_mirrored_Header 8X2A_OLogic Nexus Vault
- removed CN3, CN4: Header 2H, HDR1X2H, symbol OLogic Nexus Vault:root_0_Header 2H_OLogic Nexus Vault
- removed CN5: Header 5X2A, HDR2X5_CEN, symbol OLogic Nexus Vault:root_0_Header 5X2A_OLogic Nexus Vault
- removed D1, D3: B340A, DO-214AC, symbol OLogic Nexus Vault:root_1_SK36A-LTP_OLogic Nexus Vault
- removed D2: 1N4448W-E3-18, SOD123, symbol OLogic Nexus Vault:root_2_1N4448W-E3-18_OLogic Nexus Vault
- removed FB1: 300 Ohm @ 100MHz, 0805, RESC0805(2012)_N, symbol OLogic Nexus Vault:root_0_OL_Ferrite_OLogic Nexus Vault
- removed L1: SSR1028 6.8uH, SRU1028, symbol OLogic Nexus Vault:root_0_SSR1028_OLogic Nexus Vault
- removed L2: SSR1210 100uH, SRR1210, symbol OLogic Nexus Vault:root_0_SSR1210_OLogic Nexus Vault
- removed LED1: 0603 LED, SM-LED-0603, symbol OLogic Nexus Vault:root_3_LED_SINGLE_GENERIC_OLogic Nexus Vault
- removed LED3: G, SM-LED-0603, symbol OLogic-Diode-Opto-LED:root_3_0603 LED_OLogic-Diode-Opto-LED.IntLib
- removed PWR_OUT1: TestPoint_BLK, TestPoint-TH 42 mil, symbol OLogic Nexus Vault:root_0_TestPoint_BLK_OLogic Nexus Vault
- removed Q1, Q2: MMBT2907A, SOT23, symbol OLogic Nexus Vault:root_0_mirrored_MMBT2907A_OLogic Nexus Vault
- removed Q3, Q4: MMBT3904, SOT23, symbol OLogic-Trans-Drivers:root_0_MMBT3904_OLogic-Trans-Drivers.IntLib
- removed Q5, Q6: BSS123TA, SOT23-3L, symbol OLogic Nexus Vault:root_0_mirrored_BSS123TA_OLogic Nexus Vault
- removed R1: 33K, RESC0603(1608)_N, symbol OLogic Nexus Vault:root_3_=Resistance_OLogic Nexus Vault
- removed R10, R16, R21, R23: 1.0K, RESC0603(1608)_N, symbol OLogic Nexus Vault:root_3_=Resistance_OLogic Nexus Vault
- removed R11, R17, R24: 10K, RESC0603(1608)_N, symbol OLogic Nexus Vault:root_0_=Resistance_OLogic Nexus Vault
- removed R12, R19, R20: 1.0K, RESC0603(1608)_N, symbol OLogic Nexus Vault:root_0_=Resistance_OLogic Nexus Vault
- removed R13, R2, R26, R27, R3, R4, R7: 10K, RESC0603(1608)_N, symbol OLogic Nexus Vault:root_3_=Resistance_OLogic Nexus Vault
- removed R15: 100K, RESC0603(1608)_N, symbol OLogic Nexus Vault:root_0_=Resistance_OLogic Nexus Vault
- removed R18: 1.0K, RESC0603(1608)_N, symbol OLogic Nexus Vault:root_1_=Resistance_OLogic Nexus Vault
- removed R22: 0.33, RESC1206(3216)_N, symbol OLogic Nexus Vault:root_0_=Resistance_OLogic Nexus Vault
- removed R25: 100, RESC0603(1608)_N, symbol OLogic Nexus Vault:root_0_=Resistance_OLogic Nexus Vault
- removed R28: 100, RESC0603(1608)_N, symbol OLogic Nexus Vault:root_3_=Resistance_OLogic Nexus Vault
- removed R29, R31, R32: 10K, RESC0603(1608)_M, symbol OLogic Nexus Vault:root_0_=Resistance_OLogic Nexus Vault
- removed R5: 10K, RESC0603(1608)_L, symbol OLogic Nexus Vault:root_3_=Resistance_OLogic Nexus Vault
- removed R6, R8, R9: 10k, RESC0603(1608)_M, symbol OLogic Nexus Vault:root_0_=Resistance_OLogic Nexus Vault
- removed U1: ~, TO-252_N, symbol OLogic Nexus Vault:root_0_PM-REG-LD29150-SOT3_OLogic Nexus Vault
- removed U10: TPS7A4515KTTR, TPS7A4515KTTR, symbol hdmi_lvds:root_0_TPS7A4515KTTR_hdmi_lvds.IntLib
- removed U11: OPA2320, SOIC-8_NoPad, symbol OLogic Nexus Vault:root_0_mirrored_OPA2320_OLogic Nexus Vault
- removed U12, U6: OPA2320, SOIC-8_NoPad, symbol OLogic Nexus Vault:root_0_OPA2320_OLogic Nexus Vault
- removed U13: INA219, INA219, symbol hdmi_lvds:root_0_INA219_hdmi_lvds.IntLib
- removed U14: INA180A1, SOT-23-5_MC, symbol hdmi_lvds:root_0_INA180A1_hdmi_lvds.IntLib
- removed U15: LM334, LM334, symbol hdmi_lvds:root_0_LM334_hdmi_lvds.IntLib
- removed U2: mcp4728, MCP4728, symbol hdmi_lvds:root_0_mcp4728_hdmi_lvds.IntLib
- removed U3: TPS54331, TPS54331, symbol hdmi_lvds:root_0_TPS54331_hdmi_lvds.IntLib
- removed U4: mcp9808, 8MSOP, symbol hdmi_lvds:root_0_mcp9808_hdmi_lvds.IntLib
- removed U5: LD1117S33, DSO-G3, symbol OLogic Nexus Vault:root_0_LD1117S33_OLogic Nexus Vault
- removed U7: TCA9534APWR, TCA9534APWR-Footprint-1, symbol OLogic Nexus Vault:root_0_TCA9534APWR_OLogic Nexus Vault
- removed U8: LM2776, SOt-23-6, symbol *:root_0_LM2776_*
- removed U9: OPA2320, SOIC-8_NoPad, symbol OLogic Nexus Vault:root_2_mirrored_OPA2320_OLogic Nexus Vault
- added C1: 100pf, Capacitor_SMD:C_0603_1608Metric_Pad1.08x0.95mm_HandSolder, symbol Device:C_Small
- added C10, C11, C18, C22, C25, C27, C30, C43, C45, C53, C6, C8, C9: 10uF, Capacitor_SMD:C_0603_1608Metric_Pad1.08x0.95mm_HandSolder, symbol Device:C_Small
- added C12, C13, C14, C16, C19, C2, C20, C21, C23, C26, C3, C31, C32, C36, C4, C42, C44, C47, C5, C7: 0.1uF, Capacitor_SMD:C_0603_1608Metric_Pad1.08x0.95mm_HandSolder, symbol Device:C_Small
- added C15: 0.1uf, Capacitor_SMD:C_0603_1608Metric_Pad1.08x0.95mm_HandSolder, symbol Device:C_Small
- added C17, C34: 4.7uF, Capacitor_SMD:C_1206_3216Metric_Pad1.33x1.80mm_HandSolder, symbol Device:C_Small
- added C24, C46, C50: 1uF, Capacitor_SMD:C_0603_1608Metric_Pad1.08x0.95mm_HandSolder, symbol Device:C_Small
- added C33: 0.01uf, Capacitor_SMD:C_0603_1608Metric_Pad1.08x0.95mm_HandSolder, symbol Device:C_Small
- added C37, C38: 47uF, Capacitor_SMD:C_1206_3216Metric_Pad1.33x1.80mm_HandSolder, symbol Device:C_Small
- added C39: 0.01uF, Capacitor_SMD:C_0603_1608Metric_Pad1.08x0.95mm_HandSolder, symbol Device:C_Small
- added C40: 150pf, Capacitor_SMD:C_0603_1608Metric_Pad1.08x0.95mm_HandSolder, symbol Device:C_Small
- added C41: 8.2nf, Capacitor_SMD:C_0603_1608Metric_Pad1.08x0.95mm_HandSolder, symbol Device:C_Small
- added CN1: PWR Conn, Connector_PinHeader_2.54mm:PinHeader_2x05_P2.54mm_Vertical, symbol Connector_Generic:Conn_02x05_Top_Bottom
- added CN2: Header 8x2A, symbol Connector_Generic:Conn_02x08_Top_Bottom
- added CN3, CN4, CN5: SW_BPASSS, Connector_PinHeader_2.54mm:PinHeader_1x02_P2.54mm_Horizontal, symbol Connector_Generic:Conn_01x02
- added D1, D3: B340, Diode_SMD:D_SMC, symbol Diode:B340
- added D2: 1N4448, Diode_SMD:Nexperia_CFP3_SOD-123W, symbol Diode:1N4448
- added FB1: 300 Ohm @ 100MHz, 0805, symbol Device:FerriteBead
- added I2C_SCL1: I2C_SCL, TestPoint:TestPoint_THTPad_D2.0mm_Drill1.0mm, symbol Connector:TestPoint
- added I2C_SCL2: GND, TestPoint:TestPoint_THTPad_D2.0mm_Drill1.0mm, symbol Connector:TestPoint
- added I2C_SDA1: I2C_SDA, TestPoint:TestPoint_THTPad_D2.0mm_Drill1.0mm, symbol Connector:TestPoint
- added I_sample1, I_sample10, I_sample11, I_sample12, I_sample2, I_sample6, I_sample7, I_sample8, I_sample9, OSA_TP2, OSA_TP3, OSA_TP4, REG_IN2: TP2, TestPoint:TestPoint_THTPad_D2.0mm_Drill1.0mm, symbol Connector:TestPoint
- added I_sample13: Spare_1, TestPoint:TestPoint_THTPad_D2.0mm_Drill1.0mm, symbol Connector:TestPoint
- added L1: 6.8uH, Inductor_SMD:L_TDK_SLF12565, symbol Device:L_Ferrite_Small
- added L2: 100uH, Inductor_SMD:L_TDK_SLF12565, symbol Device:L_Ferrite_Small
- added LED1: LED, LED_SMD:LED_0603_1608Metric, symbol Device:LED
- added LED2: LED2, LED_SMD:LED_0603_1608Metric, symbol Device:LED
- added PWR_OUT1: PWR_OUT1, TestPoint:TestPoint_THTPad_D2.0mm_Drill1.0mm, symbol Connector:TestPoint
- added Q1, Q5: MMBT3906, Package_TO_SOT_SMD:SOT-23, symbol Transistor_BJT:MMBT3906
- added Q2, Q3: MMBT3904, Package_TO_SOT_SMD:SOT-23, symbol lps_regulator:MMBT3904
- added Q4, Q6: BSS123, Package_TO_SOT_SMD:SOT-23, symbol Transistor_FET:BSS123
- added R1, R22: 100R, Resistor_SMD:R_0603_1608Metric_Pad0.98x0.95mm_HandSolder, symbol Device:R_Small_US
- added R10, R11: 10R, Resistor_SMD:R_0603_1608Metric_Pad0.98x0.95mm_HandSolder, symbol Device:R_Small_US
- added R12, R17, R19, R5, R9: 1K, Resistor_SMD:R_0603_1608Metric_Pad0.98x0.95mm_HandSolder, symbol Device:R_Small_US
- added R13, R14, R15, R16, R20, R23, R27, R28, R29, R30, R4, R6, R7, R8: 10K, Resistor_SMD:R_0603_1608Metric_Pad0.98x0.95mm_HandSolder, symbol Device:R_Small_US
- added R18, R2: 33K, Resistor_SMD:R_0603_1608Metric_Pad0.98x0.95mm_HandSolder, symbol Device:R_Small_US
- added R21: 51K, Resistor_SMD:R_0603_1608Metric_Pad0.98x0.95mm_HandSolder, symbol Device:R_Small_US
- added R25, R32: 1K, Resistor_SMD:R_0805_2012Metric_Pad1.20x1.40mm_HandSolder, symbol Device:R_Small_US
- added R26: 5.1K, Resistor_SMD:R_0603_1608Metric_Pad0.98x0.95mm_HandSolder, symbol Device:R_Small_US
- added R3: 0.1R, Resistor_SMD:R_1206_3216Metric_Pad1.30x1.75mm_HandSolder, symbol Device:R_Small_US
- added REG_IN1: REG_IN1, TestPoint:TestPoint_THTPad_D2.0mm_Drill1.0mm, symbol Connector:TestPoint
- added U1: TPS7A4515KTTR, Package_TO_SOT_SMD:TO-263-5_TabPin3, symbol jerrys_Library:TPS7A4515KTTR
- added U10: LM78M05_TO252, Package_TO_SOT_SMD:TO-252-2, symbol Regulator_Linear:LM78M05_TO252
- added U11: LD1117S33TR_SOT223, Package_TO_SOT_SMD:SOT-223-3_TabPin2, symbol Regulator_Linear:LD1117S33TR_SOT223
- added U12: LM2776, Package_TO_SOT_SMD:SOT-23-6, symbol Regulator_SwitchedCapacitor:LM2776
- added U14: TPS54331, Package_SO:SOIC-8-1EP_3.9x4.9mm_P1.27mm_EP2.29x3mm_ThermalVias, symbol jerrys_Library:root_0_TPS54331_hdmi_lvds.IntLib
- added U2: INA180A1, Package_TO_SOT_SMD:SOT-23-5, symbol Amplifier_Current:INA180A1
- added U3: INA219AxD, Package_SO:SOIC-8_3.9x4.9mm_P1.27mm, symbol Sensor_Energy:INA219AxD
- added U4, U9: OPA2320, Package_SO:SOIC-8_3.9x4.9mm_P1.27mm, symbol lps_regulator_rev_12-altium-import:root_0_mirrored_OPA2320_OLogic Nexus Vault
- added U5: LM334, Package_SO:SOIC-8_3.9x4.9mm_P1.27mm, symbol jerrys_Library:LM334
- added U6: MCP9808, Package_SO:MSOP-8_3x3mm_P0.65mm, symbol Sensor_Temperature:MCP9808_MSOP
- added U7: MCP4728, Package_SO:MSOP-10_3x3mm_P0.5mm, symbol Analog_DAC:MCP4728
- added U8: TCA9534, Package_SO:SOIC-16W_7.5x10.3mm_P1.27mm, symbol Interface_Expansion:TCA9534
- C29: renamed from C47; value o.1uF -> 0.1uF; footprint Capacitor_SMD:C_0805_2012Metric_Pad1.18x1.45mm_HandSolder -> Capacitor_SMD:C_0603_1608Metric_Pad1.08x0.95mm_HandSolder
- renumbered D5 to LED3, R30 to R24, R14 to R31
Connections:
- net +3V3: now also C14.1, C15.1, C16.1, C18.2, C2.1, C23.2, C7.1, I_sample12.1, R15.1, R19.1, R25.2, R28.1, R6.2, R7.2, U11.2 (VO), U2.5 (V+), U3.5 (VS), U6.8 (V_{DD}), U7.1 (VDD), U8.16 (VDD)
- net +5V0: now also C21.2, C22.2, C25.2, C27.2, I_sample11.1, U10.3 (VO), U11.3 (VI), U12.3 (VIN), U12.4 (EN)
- net +VIN_SW: now also C17.1, C19.1, C24.2, C33.1, C34.1, C4.1, CN2.13 (Pin_13), CN2.14 (Pin_14), CN2.5 (Pin_5), CN2.6 (Pin_6), CN3.1 (Pin_1), I_sample10.1, R29.2, R5.2, U10.1 (VI), U14.2 (VIN), U4.8 (V+), U9.8 (V+)
- net /RST: now also CN2.9 (Pin_9), I_sample6.1
- net Current_Limit: now also CN2.3 (Pin_3), LED2.1 (K), Q2.3 (C), U8.4 (P0)
- net Debug_LED: now also U8.6 (P2)
- net GND: now also C10.2, C11.2, C12.2, C13.2, C14.2, C15.2, C16.2, C17.2, C18.1, C19.2, C2.2, C20.2, C21.1, C22.1, C23.1, C24.1, C25.1, C26.1, C27.1, C3.2, C32.1, C33.2, C34.2, C37.2, C38.2, C39.2, C4.2, C41.2, C42.2, C43.1, C44.2, C45.2, C46.2, C5.1, C53.1, C6.2, C7.2, C8.2, C9.2, CN1.10 (Pin_10), CN1.4 (Pin_4), CN1.5 (Pin_5), CN1.9 (Pin_9), CN2.15 (Pin_15), CN2.16 (Pin_16), CN2.7 (Pin_7), CN2.8 (Pin_8), CN4.2 (Pin_2), CN5.2 (Pin_2), D1.2 (A), D3.2 (A), I2C_SCL2.1, I_sample7.1, I_sample8.1, I_sample9.1, LED1.1 (K), Q2.2 (E), Q4.2 (S), Q6.2 (S), R13.2, R18.1, R20.2, R22.2, R27.1, R32.1, U10.2 (GND), U11.1 (GND), U12.2 (GND), U14.7 (GND), U14.9 (PPAD), U2.2 (GND), U3.1 (A1), U3.2 (A0), U3.6 (GND), U6.4 (GND), U6.5 (A2), U6.6 (A1), U6.7 (A0), U7.10 (VSS), U7.4 (~{LDAC}), U8.1 (A0), U8.2 (A1), U8.3 (A2), U8.8 (GND), U9.5 (INB+)
- net I2C_SCL: now also CN2.1 (Pin_1), I2C_SCL1.1, R6.1, U3.4 (SCL), U6.2 (SCL), U7.2 (SCL), U8.15 (SDA)
- net I2C_SDA: now also CN2.2 (Pin_2), I2C_SDA1.1, R7.1, U3.3 (SDA), U6.1 (SDA), U7.3 (SDA), U8.14 (SCL)
- net IA_TP: now also OSA_TP3.1, R17.2, U7.7 (VOUTB)
- net I_Sample: now also C6.1, CN2.11 (Pin_11), I_sample1.1, R23.1, U4.5 (INB+)
- net OUTPUT_ENB: now also CN2.4 (Pin_4), Q6.1 (G), R20.1, U8.5 (P1)
- net Pwr_Out: now also C3.1, C8.1, C9.1, CN1.1 (Pin_1), CN1.2 (Pin_2), CN1.6 (Pin_6), CN1.7 (Pin_7), D1.1 (K), PWR_OUT1.1, R1.2, R10.1, R3.1, U5.V+ (4)
- net Pwr_Out_Sample: now also C13.1, R11.1, R3.2, U1.4 (OUT)
- net VA_TP: now also OSA_TP4.1, U7.6 (VOUTA), U9.3 (INA+)
- net VA_TP_GAIN: now also C1.2, R12.1, R4.1, U9.1 (OUTA)
- net V_offset_adj: now also OSA_TP2.1, R9.1, U7.8 (VOUTC)
- net at R24.1: now also U5.1 (R)
- net -5V0 renamed -5VA
- net -5VA: now also C20.1, C26.2, C5.2, C53.2, I_sample2.1, Q1.3 (C), R32.2, U12.1 (VOUT), U4.4 (V-), U5.2 (V-), U5.3 (V-), U5.6 (V-), U5.7 (V-), U9.4 (V-)
- new net: LED1.2 (A), R25.1
- new net: CN5.1 (Pin_1), Q3.1 (B), R16.2
- new net: Q3.2 (E), R22.1
- new net: Q3.3 (C), Q4.3 (D), R12.2, U4.3 (INA+)
- new net: C36.2, D3.1 (K), L1.1, U14.8 (PH)
- new net: C32.2, C37.1, C38.1, CN3.2 (Pin_2), FB1.1, L1.2, R2.2
- new net: I_sample13.1, U7.9 (VOUTD)
- new net: C10.1, C11.1, C12.1, C43.2, C44.1, C45.1, C46.1, L2.2, REG_IN1.1, U1.1 (/SHDN), U1.2 (IN)
- new net: Q1.1 (B), U4.1 (OUTA)
- new net: C47.2, R8.1, R9.2, U4.2 (INA-)
- new net: Q5.3 (C), R27.2, U14.5 (VSENSE)
- new net: C36.1, U14.1 (BOOT)
- new net: CN4.1 (Pin_1), R29.1, U14.3 (EN)
- new net: C39.1, U14.4 (SS)
- new net: C40.1, C41.1, U14.6 (COMP)
- new net: C47.1, Q1.2 (E), R14.1, R5.1, R8.2, REG_IN2.1, U1.3 (GND), U1.6 (TAB)
- new net: D2.1 (K), Q5.2 (E), R2.1
- new net: D2.2 (A), Q5.1 (B), R14.2
- new net: C30.1, R17.1, R21.2, U4.6 (INB-)
- new net: C30.2, R16.1, R21.1, R30.1, U4.7 (OUTB)
- new net: Q2.1 (B), R30.2
- new net: R26.2, U9.6 (INB-)
- new net: R26.1, U9.7 (OUTB)
- new net: C1.1, R13.1, R4.2, U9.2 (INA-)
- new net: C31.1, R11.2, U2.3 (+), U3.8 (IN+)
- new net: Q4.1 (G), Q6.3 (D), R28.2
- new net: C40.2, R18.2
- new net: R23.2, U2.1
- new net: C31.2, R10.2, U2.4 (-), U3.7 (IN-)
- new net: C50.1, U12.6 (C1-)
- new net: C50.2, U12.5 (C1+)
- new net: C42.1, FB1.2, L2.1
- new net: LED2.2 (A), R19.2
- new net: CN1.3 (Pin_3), CN1.8 (Pin_8), R1.1, U1.5 (SENSE)
- new net /INT: CN2.10 (Pin_10), R15.2, U8.13 (~{INT})
- no-connect marks 11 -> 10
Other:
- note added: "+5V1"
- note added: "+VIN_SW1"
- note added: "1206"
- note added: "3V1"
- note added: "IA_TP1"
- note added: "I_sample1"
- note added: "OSA_TP1"
- note added: "REG_IN1"
- note added: "TPS7A4515KTTR"
- note added: "VA_TP1"
- note removed: "Lab Power Supply"
- moved on the sheet: C29, LED3, R24, R31
